Commit message: feat: rename "bioscara" macro to "bioscara_arm" to align with convention

File: lib/ros2_ws/src/dalsa_bioscara_arm/bioscara_arm_description/urdf/bioscara.urdf.xacro (robot description, xacro)
@@ -1,5 +1,5 @@
 <?xml version="1.0" ?>
 <robot xmlns:xacro="http://www.ros.org/wiki/xacro">
-  <xacro:macro name="bioscara" params="parameters prefix parent *origin">
+  <xacro:macro name="bioscara_arm" params="parameters prefix parent *origin">
     <xacro:include filename="$(find bioscara_arm_description)/urdf/materials.xacro" />
     <xacro:property name="tool_flange_zheight" value="0.135"/>

File: lib/ros2_ws/src/dalsa_bioscara_arm/bioscara_arm_description/urdf/bioscara_arm.xacro (robot description, xacro)
@@ -10,14 +10,14 @@
     <xacro:include filename="$(find bioscara_arm_description)/urdf/bioscara.urdf.xacro" />
     <xacro:include filename="$(find bioscara_arm_description)/urdf/bioscara.ros2control" />
-    <xacro:bioscara_ros2_control
+    <xacro:bioscara_arm_ros2_control
       prefix="${prefix}"
       parameters="${params}"
       use_mock_hardware="${use_mock_hardware}"/>
-    <xacro:bioscara
+    <xacro:bioscara_arm
       parent="${parent}"
       prefix="${prefix}"
       parameters="${params}">
       <xacro:insert_block name="origin" />
-    </xacro:bioscara>
+    </xacro:bioscara_arm>
   </xacro:macro>
 </robot>
